File: Logic.sch (KiCad schematic (older format))
At the start: 13 parts, among them J902 I2C, J904 ISP, U901 ATMEGA328P-AU, Y901 16M

Commit message: switching to more convenient notation of values, e.g. 100K instead of 0M1
Parts:
- C901, C902, C903: value 0u1 -> 100n
- R904, R905: value 4k7 -> 4K7
Changed lines of the file:
@@
 P 1550 2000
 F 0 "C903" H 1560 2070 50  0000 L CNN
-F 1 "0u1" H 1560 1920 50  0000 L CNN
+F 1 "100n" H 1560 1920 50  0000 L CNN
 F 2 "Capacitors_SMD:C_0805_HandSoldering" H 1550 2000 50  0001 C CNN
 F 3 "" H 1550 2000 50  0001 C CNN
@@
 P 1200 2000
 F 0 "C902" H 1210 2070 50  0000 L CNN
-F 1 "0u1" H 1210 1920 50  0000 L CNN
+F 1 "100n" H 1210 1920 50  0000 L CNN
 F 2 "Capacitors_SMD:C_0805_HandSoldering" H 1200 2000 50  0001 C CNN
 F 3 "" H 1200 2000 50  0001 C CNN
@@
 P 850 2000
 F 0 "C901" H 860 2070 50  0000 L CNN
-F 1 "0u1" H 860 1920 50  0000 L CNN
+F 1 "100n" H 860 1920 50  0000 L CNN
 F 2 "Capacitors_SMD:C_0805_HandSoldering" H 850 2000 50  0001 C CNN
 F 3 "" H 850 2000 50  0001 C CNN
@@
 P 8200 2500
 F 0 "R905" H 8230 2520 50  0000 L CNN
-F 1 "4k7" H 8230 2460 50  0000 L CNN
+F 1 "4K7" H 8230 2460 50  0000 L CNN
 F 2 "Resistors_SMD:R_0805_HandSoldering" H 8200 2500 50  0001 C CNN
 F 3 "" H 8200 2500 50  0001 C CNN
@@
 P 7900 2500
 F 0 "R904" H 7930 2520 50  0000 L CNN
-F 1 "4k7" H 7930 2460 50  0000 L CNN
+F 1 "4K7" H 7930 2460 50  0000 L CNN
 F 2 "Resistors_SMD:R_0805_HandSoldering" H 7900 2500 50  0001 C CNN
 F 3 "" H 7900 2500 50  0001 C CNN
