File: RTC.sch (KiCad schematic (older format))
At the start: 8 parts, among them U1002 DS3231MZ, U1003 FM24C04A, U1004 DCF1

Commit message: switching to more convenient notation of values, e.g. 100K instead of 0M1
Parts:
- C1002, C1003: value 0u1 -> 100n
Changed lines of the file:
@@
 P 2650 1750
 F 0 "C1002" V 2750 1750 50  0000 L CNN
-F 1 "0u1" V 2550 1750 50  0000 L CNN
+F 1 "100n" V 2550 1750 50  0000 L CNN
 F 2 "Capacitors_SMD:C_0805_HandSoldering" H 2650 1750 50  0001 C CNN
 F 3 "" H 2650 1750 50  0001 C CNN
@@
 P 2650 4800
 F 0 "C1003" H 2660 4870 50  0000 L CNN
-F 1 "0u1" H 2660 4720 50  0000 L CNN
+F 1 "100n" H 2660 4720 50  0000 L CNN
 F 2 "Capacitors_SMD:C_0805_HandSoldering" H 2650 4800 50  0001 C CNN
 F 3 "" H 2650 4800 50  0001 C CNN
