File: USB.sch (KiCad schematic (older format))
At the start: 10 parts, among them J1101 UART, J1102 USB_OTG, U1103 CH340G, Y1101 12M

Commit message: switching to more convenient notation of values, e.g. 100K instead of 0M1
Parts:
- C1101: value 0u1 -> 100n
Changed lines of the file:
@@
 P 4650 3350
 F 0 "C1101" H 4660 3420 50  0000 L CNN
-F 1 "0u1" H 4660 3270 50  0000 L CNN
+F 1 "100n" H 4660 3270 50  0000 L CNN
 F 2 "Capacitors_SMD:C_0805_HandSoldering" H 4650 3350 50  0001 C CNN
 F 3 "" H 4650 3350 50  0001 C CNN
